Commit message: file upload

File: mani_skill2/assets/descriptions/xarm_description/xarm6_with_gripper.urdf (robot description, URDF)
Before this commit: robot xarm6_with_gripper, 17 links, 16 joints
Links:
- link left_finger: geometry collision mesh filename=package://meshes/left_finger.STL; visual mesh filename=package://meshes/left_finger.STL
- link left_inner_knuckle: geometry collision mesh filename=package://meshes/left_inner_knuckle.STL; visual mesh filename=package://meshes/left_inner_knuckle.STL
- link left_outer_knuckle: geometry collision mesh filename=package://meshes/left_outer_knuckle.STL; visual mesh filename=package://meshes/left_outer_knuckle.STL
- link link1: geometry collision mesh filename=package://meshes/link1.stl; visual mesh filename=package://meshes/link1.stl
- link link2: geometry collision mesh filename=package://meshes/link2.stl; visual mesh filename=package://meshes/link2.stl
- link link3: geometry collision mesh filename=package://meshes/link3.stl; visual mesh filename=package://meshes/link3.stl
- link link4: geometry collision mesh filename=package://meshes/link4.stl; visual mesh filename=package://meshes/link4.stl
- link link5: geometry collision mesh filename=package://meshes/link5.stl; visual mesh filename=package://meshes/link5.stl
- link link6: geometry collision mesh filename=package://meshes/link6.stl; visual mesh filename=package://meshes/link6.stl
- link link_base: geometry collision mesh filename=package://meshes/base.stl; visual mesh filename=package://meshes/base.stl
- link right_finger: geometry collision mesh filename=package://meshes/right_finger.STL; visual mesh filename=package://meshes/right_finger.STL
- link right_inner_knuckle: geometry collision mesh filename=package://meshes/right_inner_knuckle.STL; visual mesh filename=package://meshes/right_inner_knuckle.STL
- link right_outer_knuckle: geometry collision mesh filename=package://meshes/right_outer_knuckle.STL; visual mesh filename=package://meshes/right_outer_knuckle.STL
- link xarm_gripper_base_link: geometry collision mesh filename=package://meshes/base_link.STL; visual mesh filename=package://meshes/base_link.STL
