Commit message: file upload

File: mani_skill2/assets/descriptions/xarm_description/xarm6_with_gripper_spoon.urdf (robot description, URDF)
Before this commit: robot xarm6_with_gripper, 18 links, 17 joints
Joints:
- joint drive_joint: limit lower=0 upper=0.85 effort=50 velocity=2 -> lower=0.85 upper=0.85 effort=50 velocity=2
- joint left_finger_joint: limit lower=0 upper=0.85 effort=50 velocity=2 -> lower=0.85 upper=0.85 effort=50 velocity=2
- joint left_finger_spoon: origin xyz=0 -0.03 0.026 rpy=-1.3531044 -1.5207655 1.6368985 -> xyz=0 -0.03 0.026 rpy=1.3531044 -1.5207655 1.6368985
- joint left_inner_knuckle_joint: limit lower=0 upper=0.85 effort=50 velocity=2 -> lower=0.85 upper=0.85 effort=50 velocity=2
- joint right_finger_joint: limit lower=0 upper=0.85 effort=50 velocity=2 -> lower=0.85 upper=0.85 effort=50 velocity=2
- joint right_inner_knuckle_joint: limit lower=0 upper=0.85 effort=50 velocity=2 -> lower=0.85 upper=0.85 effort=50 velocity=2
- joint right_outer_knuckle_joint: limit lower=0 upper=0.85 effort=50 velocity=2 -> lower=0.85 upper=0.85 effort=50 velocity=2
