Commit message: file upload

File: mani_skill2/assets/descriptions/panda_spoon.urdf (robot description, URDF)
Before this commit: robot panda, 13 links, 12 joints
Links:
- removed link panda_hand
- removed link panda_hand_tcp
- removed link panda_leftfinger
- removed link panda_rightfinger
- added link spoon, mass 0.54156; collision mesh filename=package://franka_description/meshes/spoon.STL.convex.stl scale=0.001 0.001 0.001; visual mesh filename=package://franka_description/meshes/spoon.STL scale=0.001 0.001 0.001
Joints:
- removed joint panda_finger_joint1
- removed joint panda_finger_joint2
- removed joint panda_hand_joint
- removed joint panda_hand_tcp_joint
- added joint left_finger_spoon: type fixed, parent panda_link8, child spoon, origin xyz=0 -0.03 0.026 rpy=1.3531044 -1.5207655 1.6368985
